File: Revisions/Original/Project NEO Zia Original.kicad_pcb (KiCad board)
At the start: 2 copper layers, 214.8 x 214.5 mm, 103 parts, among them J1 Conn_01x03_Pin, J2 Conn_01x03_Pin

Commit message: - Added "For more info visit: https://github.com/JZRod/Project-NEO-Zia" to all versions 	# backported to all pre-existing versions - Fixed voltage regulator tab being shorted to GND 	# Backported to all relevant rev's - Added gbr, step, and csv files to all versions (except original) - Fixed sheet information to match REVISION NOTES.txt
Other:
- board text added: "For more info visit: https://github.com/JZRod/Project-NEO-Zia"
Changed lines of the file:
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@@
 	(paper "A3")
 	(title_block
-		(date "2025-05-08")
+		(title "Project NEO Zia")
+		(date "5/12/2025")
+		(rev "Original")
+		(comment 1 "Started on 4/19/2025")
+		(comment 2 "What's left after my hard drive died")
+		(comment 3 "DO NOT USE")
 	)
 	(layers
@@
 		)
 	)
+	(gr_text "For more info visit: https://github.com/JZRod/Project-NEO-Zia"
+		(at 302.725 164.7 0)
+		(layer "B.SilkS")
+		(effects
+			(font
+				(size 1.5 1.5)
+				(thickness 0.3)
+				(bold yes)
+			)
+			(justify left bottom mirror)
+		)
+	)
