File: Revisions/REV 1.5/Project NEO Zia REV 1_5.kicad_pcb (KiCad board)
At the start: 2 copper layers, 214.8 x 214.5 mm, 103 parts, among them J1 5-147278-2, J2 5-147278-2

Commit message: - Added "For more info visit: https://github.com/JZRod/Project-NEO-Zia" to all versions 	# backported to all pre-existing versions - Fixed voltage regulator tab being shorted to GND 	# Backported to all relevant rev's - Added gbr, step, and csv files to all versions (except original) - Fixed sheet information to match REVISION NOTES.txt
Other:
- board text added: "For more info visit: https://github.com/JZRod/Project-NEO-Zia"
Changed lines of the file:
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@@
 	(title_block
 		(title "Project NEO Zia")
-		(date "2025-05-08")
+		(date "5/17/2025")
 		(rev "1.5")
 	)
@@
 		)
 	)
+	(gr_text "For more info visit: https://github.com/JZRod/Project-NEO-Zia"
+		(at 305.825 167.2 0)
+		(layer "B.SilkS")
+		(effects
+			(font
+				(size 1.5 1.5)
+				(thickness 0.3)
+				(bold yes)
+			)
+			(justify left bottom mirror)
+		)
+	)
