File: Revisions/REV 1.5/Project NEO Zia REV 1_5.kicad_sch (KiCad schematic)
At the start: 98 parts, among them J1 5-147278-2, J2 5-147278-2

Commit message: Added Gerber and STEP files Removed un-needed files Updated sheet information
Other:
- title: (none) -> Project NEO Zia
Changed lines of the file:
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@@
 	(generator_version "9.0")
 	(paper "A3")
+	(title_block
+		(title "Project NEO Zia")
+		(date "2025-5-17")
+		(rev "1.5")
+	)
 	(text "In"
 		(exclude_from_sim no)
