File: Revisions/REV 2/Project NEO Zia REV 2.kicad_pcb (KiCad board)
At the start: 2 copper layers, 217 x 216.7 mm, 103 parts, among them J1 TSM-103-02-X-SH, J2 TSM-103-02-X-SH

Commit message: - Added "For more info visit: https://github.com/JZRod/Project-NEO-Zia" to all versions 	# backported to all pre-existing versions - Fixed voltage regulator tab being shorted to GND 	# Backported to all relevant rev's - Added gbr, step, and csv files to all versions (except original) - Fixed sheet information to match REVISION NOTES.txt
Other:
- board text added: "For more info visit: https://github.com/JZRod/Project-NEO-Zia"
Changed lines of the file:
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@@
 	(paper "A3")
 	(title_block
-		(date "2025-05-08")
+		(title "Project NEO Zia")
+		(date "5/17/2025")
+		(rev "2")
 	)
 	(layers
@@
 			(outputformat 1)
 			(mirror no)
-			(drillshape 1)
+			(drillshape 0)
 			(scaleselection 1)
-			(outputdirectory "")
+			(outputdirectory "./")
 		)
 	)
@@
 		)
 	)
+	(gr_text "For more info visit: https://github.com/JZRod/Project-NEO-Zia"
+		(at 298.875 173.025 0)
+		(layer "B.SilkS")
+		(effects
+			(font
+				(size 1.5 1.5)
+				(thickness 0.3)
+				(bold yes)
+			)
+			(justify left bottom mirror)
+		)
+	)
