File: Revisions/REV 4/Project NEO Zia REV 4.kicad_sch (KiCad schematic)
At the start: 98 parts, among them J1 TSM-103-02-L-SH-LC, J2 TSM-103-02-L-SH-LC

Commit message: - Added "For more info visit: https://github.com/JZRod/Project-NEO-Zia" to all versions 	# backported to all pre-existing versions - Fixed voltage regulator tab being shorted to GND 	# Backported to all relevant rev's - Added gbr, step, and csv files to all versions (except original) - Fixed sheet information to match REVISION NOTES.txt
Other:
- title: (none) -> Project NEO Zia
Changed lines of the file:
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@@
 	(generator_version "9.0")
 	(paper "A3")
+	(title_block
+		(title "Project NEO Zia")
+		(date "5/20/2025")
+		(rev "4")
+	)
 	(text "In"
 		(exclude_from_sim no)
