File: Revisions/REV 5/Project NEO Zia REV 5.kicad_pcb (KiCad board)
At the start: 2 copper layers, 217 x 216.7 mm, 104 parts, among them J1 TSM-103-02-L-SH-LC, J2 TSM-103-02-L-SH-LC

Commit message: - Added "For more info visit: https://github.com/JZRod/Project-NEO-Zia" to all versions 	# backported to all pre-existing versions - Fixed voltage regulator tab being shorted to GND 	# Backported to all relevant rev's - Added gbr, step, and csv files to all versions (except original) - Fixed sheet information to match REVISION NOTES.txt
Other:
- board text added: "For more info visit: https://github.com/JZRod/Project-NEO-Zia"
Changed lines of the file:
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@@
 	(paper "A3")
 	(title_block
-		(date "2025-05-08")
+		(date "5/26/2025")
 	)
 	(layers
@@
 		)
 	)
+	(gr_text "For more info visit: https://github.com/JZRod/Project-NEO-Zia"
+		(at 231.8 226.9 270)
+		(layer "B.SilkS")
+		(effects
+			(font
+				(size 1.5 1.5)
+				(thickness 0.3)
+				(bold yes)
+			)
+			(justify left bottom mirror)
+		)
+	)
