File: Revisions/REV 7.5.2/Project NEO Zia REV 7_5_2.kicad_pcb (KiCad board)
At the start: 2 copper layers, 220.2 x 220.2 mm, 149 parts, among them J1 TSM-103-02-L-SH-LC, J2 TSM-103-02-L-SH-LC, J3 Conn_01x02, U2 LM1084IS-5.0_NOPB

Commit message: - Added "For more info visit: https://github.com/JZRod/Project-NEO-Zia" to all versions 	# backported to all pre-existing versions - Fixed voltage regulator tab being shorted to GND 	# Backported to all relevant rev's - Added gbr, step, and csv files to all versions (except original) - Fixed sheet information to match REVISION NOTES.txt
Connections:
- U2 pad 4: GND -> +5V
Other:
- board text added: "For more info visit: https://github.com/JZRod/Project-NEO-Zia"
Changed lines of the file:
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@@
 	(paper "A3")
 	(title_block
-		(date "2025-10-25")
+		(title "Project NEO Zia")
+		(date "10/7/2025")
+		(rev "7.5.2")
 	)
 	(layers
@@
 			(drillshape 0)
 			(scaleselection 1)
-			(outputdirectory "C:/Users/Joshua Rodriguez/Downloads/NEO Zia/")
+			(outputdirectory "./")
 		)
 	)
@@
 			(size 7.62 10.84)
 			(layers "F.Cu" "F.Mask")
-			(net 2 "GND")
+			(net 4 "+5V")
 			(pinfunction "GND")
 			(pintype "input")
@@
 		)
 	)
+	(gr_text "For more info visit: https://github.com/JZRod/Project-NEO-Zia"
+		(at 172.45 119.35 0)
+		(layer "B.SilkS")
+		(effects
+			(font
+				(size 1.5 1.5)
+				(thickness 0.3)
+				(bold yes)
+			)
+			(justify left bottom mirror)
+		)
+	)
